Commit message: explicit configuration of moveit + ros2_control (instead of automatic moveit one)

File: src/so_arm_description/urdf/so_arm_urdf.urdf (robot description, URDF)
Before this commit: robot so_arm_urdf, 7 links, 6 joints
Links:
- link Base: geometry collision mesh filename=package://so_arm_description/meshes/Base.STL; visual mesh filename=package://so_arm_description/meshes/Base.STL
- link Fixed_Jaw: geometry collision mesh filename=package://so_arm_description/meshes/Fixed_Jaw.STL; visual mesh filename=package://so_arm_description/meshes/Fixed_Jaw.STL
- link Lower_Arm: geometry collision mesh filename=package://so_arm_description/meshes/Lower_Arm.STL; visual mesh filename=package://so_arm_description/meshes/Lower_Arm.STL
- link Moving_Jaw: geometry collision mesh filename=package://so_arm_description/meshes/Moving_Jaw.STL; visual mesh filename=package://so_arm_description/meshes/Moving_Jaw.STL
- link Rotation_Pitch: geometry collision mesh filename=package://so_arm_description/meshes/Rotation_Pitch.STL; visual mesh filename=package://so_arm_description/meshes/Rotation_Pitch.STL
- link Upper_Arm: geometry collision mesh filename=package://so_arm_description/meshes/Upper_Arm.STL; visual mesh filename=package://so_arm_description/meshes/Upper_Arm.STL
- link Wrist_Pitch_Roll: geometry collision mesh filename=package://so_arm_description/meshes/Wrist_Pitch_Roll.STL; visual mesh filename=package://so_arm_description/meshes/Wrist_Pitch_Roll.STL

File: src/so_arm_moveit_config/config/so_arm_urdf.ros2_control.xacro (robot description, xacro)
@@ -1,5 +1,5 @@
 <?xml version="1.0"?>
 <robot xmlns:xacro="http://www.ros.org/wiki/xacro">
-    <xacro:macro name="so_arm_urdf_ros2_control" params="name initial_positions_file">
+    <xacro:macro name="so_arm_description_ros2_control" params="name initial_positions_file">
         <xacro:property name="initial_positions" value="${load_yaml(initial_positions_file)['initial_positions']}"/>
         <ros2_control name="${name}" type="system">
@@ -7,5 +7,6 @@
                 <!-- By default, set up controllers for simulation. This won't work on real hardware -->
                 <!-- plugin>mock_components/GenericSystem</plugin -->
-                <plugin>topic_based_ros2_control/TopicBasedSystem</plugin>
+                <plugin>mock_components/GenericSystem</plugin>
+                <!-- <plugin>topic_based_ros2_control/TopicBasedSystem</plugin> -->
                 <param name="joint_commands_topic">/isaac_joint_commands</param>
                 <param name="joint_states_topic">/isaac_joint_states</param>

File: src/so_arm_moveit_config/config/so_arm_urdf.urdf.xacro (robot description, xacro)
@@ -3,7 +3,7 @@
     <xacro:arg name="initial_positions_file" default="initial_positions.yaml" />
     <!-- Import so_arm_urdf urdf file -->
-    <xacro:include filename="$(find so_arm_urdf)/urdf/so_arm_urdf.urdf" />
+    <xacro:include filename="$(find so_arm_description)/urdf/so_arm_urdf.urdf" />
     <!-- Import control_xacro -->
-    <xacro:include filename="so_arm_urdf.ros2_control.xacro" />
-    <xacro:so_arm_urdf_ros2_control name="FakeSystem" initial_positions_file="$(arg initial_positions_file)"/>
+    <xacro:include filename="$(find so_arm_moveit_config)/config/so_arm_urdf.ros2_control.xacro" />
+    <xacro:so_arm_description_ros2_control name="FakeSystem" initial_positions_file="$(arg initial_positions_file)"/>
 </robot>
